File: Luka One試作機.kicad_pcb (KiCad board)
At the start: 2 copper layers, 180 x 100 mm, 63 parts, among them J1 USB_C_Receptacle_USB2.0, J2 Conn_01x04_Male, U1 Pico, U2 SN74LV1T34DBV

Commit message: fix
Parts:
- added G***: LOGO, Icon:KADOYU, F.Cu at (215.8, 122.1)
Connections:
- Kailh PG1354 pad 1: (no net) -> /RB
- Kailh PG1354 pad 2: (no net) -> GND

Commit message: fix
Parts:
- R3, R4: moved to F.Cu
- moved R3 3.30 mm to (148.3, 43.0)
- moved R4 2.98 mm to (146.2, 43.0)
Connections:
- Kailh PG1354 pad 1: (no net) -> /LB
- Kailh PG1354 pad 2: (no net) -> GND
Routing:
- net /3V3: track 39.5 -> 36.6 mm, vias 0 -> 1
- net /SCL: track 16.7 -> 15.3 mm, vias 0 -> 1
- net /SDA: track 12.0 -> 10.8 mm, vias 0 -> 1
